Commit message: Refactor tbot URDF and Gazebo configurations: streamline accessory links, update sensor parameters for depth camera and laser, and adjust launch file for improved topic remapping and performance.

File: ros2_ws/src/tbot/tbot_description/urdf/accessories.urdf.xacro (robot description, xacro)
@@ -2,16 +2,9 @@
 <robot xmlns:xacro="http://ros.org/wiki/xacro">
   <!-- accessories -->
-  <link name="imu_link">
-    <!-- <visual>
-      <geometry>
-          <box size="0.036 0.039 0.005"/>
-      </geometry>
-      <material name="yellow"/>
-    </visual> -->
-  </link>
+  <link name="imu_link"></link>
   <joint name="imu_joint" type="fixed">
     <parent link="chassis_link"/>
     <child link="imu_link"/>
-    <origin xyz="${0.025-chassis_length/2} 0 ${chassis_height/2 + 0.01}" rpy="0 0 0"/>
+    <origin xyz="0 0 0" rpy="0 0 0"/>
   </joint>
   <!-- depth camera -->
@@ -42,6 +35,12 @@
       <origin xyz="0 0 0" rpy="${-pi/2} 0 ${-pi/2}"/>
   </joint>
+  <link name="camera_depth_link"></link>
+  <joint name="camera_depth_joint" type="fixed">
+      <parent link="camera_link"/>
+      <child link="camera_depth_link"/>
+      <origin xyz="0 0 0" rpy="${-pi/2} 0 ${-pi/2}"/>
+  </joint>
   <!-- lidar -->
-  <link name="laser_link">
+  <link name="base_scan">
     <visual>
       <geometry>
@@ -67,7 +66,7 @@
   </link>
   <joint name="laser_joint" type="fixed">
-    <origin xyz="${0.05} 0 ${0.1}" rpy="0 0 0"/>
+    <origin xyz="0 0 0.1" rpy="0 0 0"/>
     <parent link="chassis_link"/>
-    <child link="laser_link"/>
+    <child link="base_scan"/>
   </joint>
 </robot>
