Commit message: Update tbot configuration: add map saving command to temp script, remove obsolete Gazebo frame files, and clean up URDF and YAML configurations for improved clarity and performance.

File: ros2_ws/src/tbot/tbot_description/urdf/temp/accessories.urdf.xacro (robot description, xacro)
@@ -66,5 +66,5 @@
   </link>
   <joint name="laser_joint" type="fixed">
-    <origin xyz="0 0 0.1" rpy="0 0 0"/>
+    <origin xyz="0 0 0.135" rpy="0 0 0"/>
     <parent link="chassis_link"/>
     <child link="base_scan"/>

File: ros2_ws/src/tbot/tbot_description/urdf/temp2/tbot.urdf copy.xacro (robot description, xacro)
@@ -1,6 +1,9 @@
 <?xml version="1.0" ?>
 <robot name="tbot" xmlns:xacro="http://ros.org/wiki/xacro">
+  <xacro:arg name="is_sim" default="true"/>
   <xacro:include filename="inertial_macros.xacro"/>
-  <xacro:include filename="tbot.gazebo.xacro"/>
+  <xacro:if value="$(arg is_sim)">
+    <xacro:include filename="tbot.gazebo.xacro"/>
+  </xacro:if>
   <link name="base_footprint"/>
   <joint name="base_joint" type="fixed">
@@ -87,5 +90,7 @@
       </xacro:inertial_cylinder>
     </link>
-    <xacro:gazebo_wheel_params prefix="${prefix}"/>
+    <xacro:if value="$(arg is_sim)">
+      <xacro:gazebo_wheel_params prefix="${prefix}"/>
+    </xacro:if>
   </xacro:macro>
   <xacro:tbot_wheel prefix="left" y_offset="0.144"/>
@@ -113,5 +118,7 @@
       </xacro:inertial_sphere>
     </link>
-    <xacro:gazebo_caster_params prefix="${prefix}"/>
+    <xacro:if value="$(arg is_sim)">
+      <xacro:gazebo_caster_params prefix="${prefix}"/>
+    </xacro:if>
   </xacro:macro>
   <xacro:caster prefix="back_left" y_offset="0.064"/>
@@ -120,29 +127,18 @@
     <parent link="base_link"/>
     <child link="camera_link"/>
-    <origin xyz="-0.17 0 0.25" rpy="0 0 0"/>
+    <origin xyz="0.064 -0.065 0.094" rpy="0 0 0"/>
   </joint>
-  <link name="camera_link">
-      <visual>
-          <geometry>
-            <box size="0.02 0.095 0.02"/>
-          </geometry>
-          <material name="white"/>
-      </visual>
-      <visual>
-        <origin xyz="0 0 -0.1"/>
-        <geometry>
-            <cylinder radius="0.01" length="0.2"/>
-        </geometry>
-        <material name="black"/>
-      </visual>
-  </link>
+  <link name="camera_link"/>
   <joint name="camera_depth_rgb_joint" type="fixed">
     <parent link="camera_link"/>
-    <child link="camera_depth_rgb_link"/>
-    <origin xyz="0 0 0" rpy="0 0 0"/>
+    <child link="camera_depth_rgb_frame"/>
+    <origin xyz="0.005 0.018 0.013" rpy="0 0 0"/>
   </joint>
-  <link name="camera_depth_rgb_link">
+  <link name="camera_depth_rgb_frame">
+    <xacro:inertial_box mass="0.035" x="0.02" y="0.1" z="0.02">
+        <origin xyz="0 0 0" rpy="0 0 0"/>
+    </xacro:inertial_box>
   </link>
-  <!-- <joint name="camera_pole_joint" type="fixed">
+  <joint name="camera_pole_joint" type="fixed">
     <parent link="base_link"/>
     <child link="camera_pole_link"/>
@@ -166,4 +162,4 @@
       <origin xyz="0.02 0 -0.05" rpy="0 0 0"/>
     </xacro:inertial_cylinder>
-  </link> -->
+  </link>
 </robot>
